Commit message: NRI-124: backport modificiations made to SDF on to the model files

File: Atlas/resources/models/GFE/atlas_trooper.urdf (robot description, URDF)
Before this commit: robot atlas, 61 links, 60 joints
Joints:
- joint back_bkx: limit lower=-0.523599 upper=0.523599 effort=300 velocity=12 -> lower=-0.40 upper=0.40 effort=300 velocity=12

File: Atlas/resources/models/GFE/atlas_unplugged_v5_dual_robotiq_no_head.urdf (robot description, URDF)
Before this commit: robot atlas, 62 links, 61 joints
Joints:
- joint back_bkx: limit lower=-0.523599 upper=0.523599 effort=300 velocity=12 -> lower=-0.40 upper=0.40 effort=300 velocity=12

File: Atlas/resources/models/GFE/atlas_unplugged_v5_dual_robotiq_with_head.urdf (robot description, URDF)
Before this commit: robot atlas, 73 links, 72 joints
Joints:
- joint back_bkx: limit lower=-0.523599 upper=0.523599 effort=300 velocity=12 -> lower=-0.40 upper=0.40 effort=300 velocity=12

File: Atlas/resources/models/GFE/atlas_unplugged_v5_no_hands_no_head.urdf (robot description, URDF)
Before this commit: robot atlas, 36 links, 35 joints
Joints:
- joint back_bkx: limit lower=-0.523599 upper=0.523599 effort=300 velocity=12 -> lower=-0.40 upper=0.40 effort=300 velocity=12

File: Atlas/resources/models/GFE/atlas_unplugged_v5_no_hands_with_head.urdf (robot description, URDF)
Before this commit: robot atlas, 47 links, 46 joints
Joints:
- joint back_bkx: limit lower=-0.523599 upper=0.523599 effort=300 velocity=12 -> lower=-0.40 upper=0.40 effort=300 velocity=12
