Commit message: Regenerate the .sdfs using the new .URDFs. Also update Sensor information for switching IMU name back to simple name.

File: Atlas/resources/models/GFE/atlas_unplugged_v5_dual_robotiq_no_head.urdf (robot description, URDF)
Before this commit: robot atlas, 62 links, 61 joints
Joints:
- joint imu_joint: origin xyz=0.05991527603 0 -0.01415 rpy=0 0 0 -> xyz=-0.0905 -0.04 -0.0125 rpy=0 0 0

File: Atlas/resources/models/GFE/atlas_unplugged_v5_dual_robotiq_with_head.urdf (robot description, URDF)
Before this commit: robot atlas, 73 links, 72 joints
Joints:
- joint imu_joint: origin xyz=0.05991527603 0 -0.01415 rpy=0 0 0 -> xyz=-0.0905 -0.04 -0.0125 rpy=0 0 0

File: Atlas/resources/models/GFE/atlas_unplugged_v5_no_hands_no_head.urdf (robot description, URDF)
Before this commit: robot atlas, 36 links, 35 joints
Joints:
- joint imu_joint: origin xyz=0.05991527603 0 -0.01415 rpy=0 0 0 -> xyz=-0.0905 -0.04 -0.0125 rpy=0 0 0

File: Atlas/resources/models/GFE/atlas_unplugged_v5_no_hands_with_head.urdf (robot description, URDF)
Before this commit: robot atlas, 47 links, 46 joints
Joints:
- joint imu_joint: origin xyz=0.05991527603 0 -0.01415 rpy=0 0 0 -> xyz=-0.0905 -0.04 -0.0125 rpy=0 0 0
